File: design/analog_front_end.sch (KiCad schematic (older format))
At the start: 17 parts, among them U1 ACS712

Commit message: Fix #4: add GPIO to reset microcontroller from pi.
* Add a Raspeberry pi pin (GPIO 18) to reset microcontroller.
* Add a Raspebeery pi pin (GPIO 23) to control the microcontroller status.
* Add a RGB LED connected to the microcontroller (PD0, PD1, PD2).
* Rename all the sheets to PIVI v1.1.
Parts:
- C1, C22, C23, C25, C26: symbol C -> C-RESCUE-pivi-shield
- R10, R11, R12, R13, R14, R15, R16, R17, R19: symbol R -> R-RESCUE-pivi-shield

Commit message: Fix #4: Move RGB LED from microcontroller to pi.
* Move RGB LED. Now it is controlled by the raspberry pi.
* Change some new libraries for capacitors and resistors.
Parts:
- C1, C22, C23, C25, C26: symbol C-RESCUE-pivi-shield -> C
Connections:
- wire segments 31 -> 34
Changed lines of the file:
@@
 LIBS:txs0104e
 LIBS:less
-LIBS:pivi-shield-cache
 EELAYER 25 0
 EELAYER END
 $Descr A4 11693 8268
 encoding utf-8
-Sheet 5 12
+Sheet 11 12
 Title "PIVI"
 Date "mar 23 jun 2015"
@@
 $EndComp
 $Comp
-L C-RESCUE-pivi-shield C23
+L C C23
 U 1 1 5497B2A3
 P 4850 4550
@@
 Current_AD
 $Comp
-L C-RESCUE-pivi-shield C22
+L C C22
 U 1 1 5497B2AF
 P 4575 4550
@@
 $EndComp
 $Comp
-L C-RESCUE-pivi-shield C25
+L C C25
 U 1 1 5497B2E4
 P 5250 1375
@@
 $EndComp
 $Comp
-L C-RESCUE-pivi-shield C26
+L C C26
 U 1 1 5497B2EB
 P 6100 2500
@@
 	4250 4450 4250 4800
 Wire Wire Line
-	4575 4800 4575 4750
-Wire Wire Line
-	4850 4050 4850 4350
+	4575 4700 4575 4800
+Wire Wire Line
+	4850 4050 4850 4400
 Connection ~ 4850 4100
 Wire Wire Line
-	4850 4750 4850 4800
-Wire Wire Line
-	4500 2100 4650 2100
+	4850 4700 4850 4800
+Wire Wire Line
+	4500 2100 4700 2100
 Wire Wire Line
 	4575 2250 4575 2100
@@
 	5675 2750 5675 2950
 Wire Wire Line
-	2225 2900 6100 2900
+	6100 2900 2225 2900
 Wire Wire Line
 	5150 1175 5675 1175
@@
 Connection ~ 5250 1175
 Wire Wire Line
-	5250 1575 5250 1625
-Wire Wire Line
-	6100 2300 6100 2100
+	5250 1525 5250 1625
+Wire Wire Line
+	6100 2100 6100 2350
 Connection ~ 6100 2100
 Wire Wire Line
-	6100 2900 6100 2700
+	6100 2650 6100 2900
 Connection ~ 6100 2900
 $Comp
@@
 	4550 1175 4550 1075
 $Comp
-L C-RESCUE-pivi-shield C1
+L C C1
 U 1 1 54C1942B
 P 4850 2100
@@
 	0    1    1    0
 $EndComp
+Wire Wire Line
+	5250 1225 5250 1175
+Wire Wire Line
+	5000 2100 5050 2100
+Wire Wire Line
+	4575 4350 4575 4400
 $EndSCHEMATC

Commit message: Changing footprints of  audio jack3.5mm Added new footprints. Added debub uart,  reference voltage Added two extra circuits for voltage measure Moving to PIVI 2.0, added circuits for current clamps
Parts:
- removed C22: 1nF, Capacitors_SMD:C_0603, symbol C
- removed C23: 100nF, Capacitors_SMD:C_0603, symbol C
- removed R16: 11.8k, Resistors_SMD:R_0603, symbol R-RESCUE-pivi-shield
- removed R17: 3.16k, Resistors_SMD:R_0603, symbol R-RESCUE-pivi-shield
- removed U1: ACS712, SOIC_Packages:SOIC-8_3.9x4.9mm_Pitch1.27mm, symbol ACS712
- R10, R11, R12, R14, R15: symbol R-RESCUE-pivi-shield -> R
- R13: value 1k -> 10k; symbol R-RESCUE-pivi-shield -> R
- R19: value 56k -> 10k; symbol R-RESCUE-pivi-shield -> R
Connections:
- net labels removed: +5V, Current_AD, Phase_Out
- wire segments 34 -> 20
Other:
- note removed: "0.106 < Vdiv < 0.951\nViout = 0.106V when I = -20A\nViout = 0.528V when I = 0A\nViout = 0.951V when I = 20A"
- note removed: "0.5 < Viout < 4.5\nViout = 0.5V when I = -20A\nViout = 2.5V when I = 0A\nViout = 4.5V when I = 20A"
- note removed: "ACS712 datasheet in Application 4 recommends using a rectifier\ndiode when connecting Viout to an ADC. The only case where Viout can\nbe negative is when I is less than -20A. As we are protected by 20A\ncircuit breakers, Viout can never be negative so we can avoid the diodes,\nand just use a voltage divider."
- note removed: "ACS712ELCTR-20A-T"
- note removed: "Atmel App note uses a sunt R and two ADC input to measure current\nin both cycles. We don't want to use shunt resistors, instead we use Hall\nEffect current sensings ICs. We use only one AD channel per circuit.\nEach AD line can measure both cycles, as the sensor output offsets the\nvoltage to make it always positive.\n\nThis needs to be taken into account in the firmware."
- note removed: "Example resistors in DK:\n11.8k 1% 0.1W: 311-11.8KHRCT-ND\n3.16k 1% 0.1W: RHM3.16KCFCT-ND\n\n"
- note removed: "In ADC unsigned mode (single ended) Vmax = Vref * (1 - 0.05)\nWhen using Vref = 1V, Vmax = 0.95\nWe use 1V internal reference. It's a band gap reference,\nnot dependent on regulated power supply stability\n\nPlease note that AVR1631 uses differential signed mode for the current\nalso.\n\nSource: http://www.atmel.com/Images/Atmel-8032-Using-the-Atmel-AVR-XMEGA-ADC_Application-Note_AVR1300.pdf"
- note removed: "Vdiv"
- moved on the sheet: C1, C25, C26, L3, L9
