File: design/ATXMEGA128A3U.sch (KiCad schematic (older format))
At the start: 20 parts, among them IC1 ATXMEGA128A3U-A, P1 CONN_02X05, X1 32.768kHz +/-20PPM 7pF SMD

Commit message: Fix #4: add GPIO to reset microcontroller from pi.
* Add a Raspeberry pi pin (GPIO 18) to reset microcontroller.
* Add a Raspebeery pi pin (GPIO 23) to control the microcontroller status.
* Add a RGB LED connected to the microcontroller (PD0, PD1, PD2).
* Rename all the sheets to PIVI v1.1.
Parts:
- C1, C10, C2, C4, C5, C6, C7, C8: symbol C -> C-RESCUE-pivi-shield
- R3, R4, R5: symbol R -> R-RESCUE-pivi-shield
Connections:
- wire segments 113 -> 115
Changed lines of the file:
@@
 EESchema Schematic File Version 2
+LIBS:pivi-shield-rescue
 LIBS:power
 LIBS:device
@@
 LIBS:memory
 LIBS:xilinx
-LIBS:special
 LIBS:microcontrollers
 LIBS:dsp
@@
 LIBS:txs0104e
 LIBS:less
+LIBS:pivi-shield-cache
 EELAYER 25 0
 EELAYER END
@@
 Sheet 2 12
 Title "PIVI"
-Date "sáb 01 nov 2014"
-Rev "1.0"
+Date "mar 23 jun 2015"
+Rev "1.1"
 Comp "Copyright (C) LESS industries S.A. 2014,2015"
 Comment1 "Share alike attribution non-commercial 4.0"
@@
 $EndDescr
 $Comp
-L R R4
+L R-RESCUE-pivi-shield R4
 U 1 1 546F43A6
 P 8350 3700
@@
 $EndComp
 $Comp
-L R R5
+L R-RESCUE-pivi-shield R5
 U 1 1 546F43A7
 P 8350 4300
@@
 $EndComp
 $Comp
-L C C4
+L C-RESCUE-pivi-shield C4
 U 1 1 548AF338
 P 4600 1525
 AR Path="/548ADE5E/548AF338" Ref="C4"  Part="1"
 AR Path="/547008F6/548AF338" Ref="C14"  Part="1"
+AR Path="/548AF338" Ref="C14"  Part="1"
 F 0 "C14" H 4600 1625 40  0000 L CNN
 F 1 "100nF" H 4606 1440 40  0000 L CNN
@@
 PF7
 $Comp
-L C C2
+L C-RESCUE-pivi-shield C2
 U 1 1 54863967
 P 3625 4650
 AR Path="/548ADE5E/54863967" Ref="C2"  Part="1"
 AR Path="/547008F6/54863967" Ref="C12"  Part="1"
+AR Path="/54863967" Ref="C12"  Part="1"
 F 0 "C12" H 3625 4750 40  0000 L CNN
 F 1 "10pF" H 3631 4565 40  0000 L CNN
@@
 P 4600 1250
 AR Path="/548ADE5E/548F45ED" Ref="#PWR10"  Part="1"
-AR Path="/547008F6/548F45ED" Ref="#PWR09"  Part="1"
-F 0 "#PWR09" H 4650 1280 20  0001 C CNN
+AR Path="/547008F6/548F45ED" Ref="#PWR010"  Part="1"
+F 0 "#PWR010" H 4650 1280 20  0001 C CNN
 F 1 "+3.3VP" H 4600 1340 30  0000 C CNN
 F 2 "" H 4600 1250 60  0000 C CNN
@@
 P 10000 2150
 AR Path="/548ADE5E/548F468B" Ref="#PWR18"  Part="1"
-AR Path="/547008F6/548F468B" Ref="#PWR010"  Part="1"
-F 0 "#PWR010" H 10050 2180 20  0001 C CNN
+AR Path="/547008F6/548F468B" Ref="#PWR011"  Part="1"
+F 0 "#PWR011" H 10050 2180 20  0001 C CNN
 F 1 "+3.3VP" H 10000 2240 30  0000 C CNN
 F 2 "" H 10000 2150 60  0000 C CNN
@@
 P 8350 3400
 AR Path="/548ADE5E/548F4755" Ref="#PWR16"  Part="1"
-AR Path="/547008F6/548F4755" Ref="#PWR011"  Part="1"
-F 0 "#PWR011" H 8400 3430 20  0001 C CNN
+AR Path="/547008F6/548F4755" Ref="#PWR012"  Part="1"
+F 0 "#PWR012" H 8400 3430 20  0001 C CNN
 F 1 "+3.3VP" H 8350 3490 30  0000 C CNN
 F 2 "" H 8350 3400 60  0000 C CNN
@@
 P 8350 4600
 AR Path="/548ADE5E/548F499C" Ref="#PWR17"  Part="1"
-AR Path="/547008F6/548F499C" Ref="#PWR012"  Part="1"
-F 0 "#PWR012" H 8400 4630 20  0001 C CNN
+AR Path="/547008F6/548F499C" Ref="#PWR013"  Part="1"
+F 0 "#PWR013" H 8400 4630 20  0001 C CNN
 F 1 "+3.3VP" H 8350 4690 30  0000 C CNN
 F 2 "" H 8350 4600 60  0000 C CNN
@@
 $EndComp
 $Comp
-L C C1
+L C-RESCUE-pivi-shield C1
 U 1 1 548F5037
 P 3625 3950
 AR Path="/548ADE5E/548F5037" Ref="C1"  Part="1"
 AR Path="/547008F6/548F5037" Ref="C11"  Part="1"
+AR Path="/548F5037" Ref="C11"  Part="1"
 F 0 "C11" H 3625 4050 40  0000 L CNN
 F 1 "10pF" H 3631 3865 40  0000 L CNN
@@
 $EndComp
 $Comp
-L C C10
+L C-RESCUE-pivi-shield C10
 U 1 1 548F53F6
 P 7700 1525
 AR Path="/548ADE5E/548F53F6" Ref="C10"  Part="1"
 AR Path="/547008F6/548F53F6" Ref="C20"  Part="1"
+AR Path="/548F53F6" Ref="C20"  Part="1"
 F 0 "C20" H 7700 1625 40  0000 L CNN
 F 1 "100nF" H 7706 1440 40  0000 L CNN
@@
 P 7700 1300
 AR Path="/548ADE5E/548F5520" Ref="#PWR13"  Part="1"
-AR Path="/547008F6/548F5520" Ref="#PWR013"  Part="1"
-F 0 "#PWR013" H 7700 1420 20  0001 C CNN
+AR Path="/547008F6/548F5520" Ref="#PWR014"  Part="1"
+F 0 "#PWR014" H 7700 1420 20  0001 C CNN
 F 1 "+3.3VADC" H 7700 1390 30  0000 C CNN
 F 2 "" H 7700 1300 60  0000 C CNN
@@
 P 8200 2150
 AR Path="/548ADE5E/548F6C6F" Ref="#PWR15"  Part="1"
-AR Path="/547008F6/548F6C6F" Ref="#PWR014"  Part="1"
-F 0 "#PWR014" H 8250 2180 20  0001 C CNN
+AR Path="/547008F6/548F6C6F" Ref="#PWR015"  Part="1"
+F 0 "#PWR015" H 8250 2180 20  0001 C CNN
 F 1 "+3.3VP" H 8200 2240 30  0000 C CNN
 F 2 "" H 8200 2150 60  0000 C CNN
@@
 $EndComp
 $Comp
-L R R3
+L R-RESCUE-pivi-shield R3
 U 1 1 5493E749
 P 4700 2250
@@
 P 4375 2250
 AR Path="/548ADE5E/5493E84E" Ref="#PWR9"  Part="1"
-AR Path="/547008F6/5493E84E" Ref="#PWR015"  Part="1"
-F 0 "#PWR015" H 4425 2280 20  0001 C CNN
+AR Path="/547008F6/5493E84E" Ref="#PWR016"  Part="1"
+F 0 "#PWR016" H 4425 2280 20  0001 C CNN
 F 1 "+3.3VP" H 4375 2340 30  0000 C CNN
 F 2 "" H 4375 2250 60  0000 C CNN
@@
 P 3450 1300
 AR Path="/548ADE5E/54967597" Ref="#PWR7"  Part="1"
-AR Path="/547008F6/54967597" Ref="#PWR016"  Part="1"
-F 0 "#PWR016" H 3450 1150 60  0001 C CNN
+AR Path="/547008F6/54967597" Ref="#PWR017"  Part="1"
+F 0 "#PWR017" H 3450 1150 60  0001 C CNN
 F 1 "+3V3" H 3450 1440 60  0000 C CNN
 F 2 "" H 3450 1300 60  0000 C CNN
@@
 $EndComp
 $Comp
-L C C5
+L C-RESCUE-pivi-shield C5
 U 1 1 5496B0BB
 P 4925 1525
 AR Path="/548ADE5E/5496B0BB" Ref="C5"  Part="1"
 AR Path="/547008F6/5496B0BB" Ref="C15"  Part="1"
+AR Path="/5496B0BB" Ref="C15"  Part="1"
 F 0 "C15" H 4925 1625 40  0000 L CNN
 F 1 "100nF" H 4931 1440 40  0000 L CNN
@@
 $EndComp
 $Comp
-L C C6
+L C-RESCUE-pivi-shield C6
 U 1 1 5496B0F5
 P 5225 1525
 AR Path="/548ADE5E/5496B0F5" Ref="C6"  Part="1"
 AR Path="/547008F6/5496B0F5" Ref="C16"  Part="1"
+AR Path="/5496B0F5" Ref="C16"  Part="1"
 F 0 "C16" H 5225 1625 40  0000 L CNN
 F 1 "100nF" H 5231 1440 40  0000 L CNN
@@
 $EndComp
 $Comp
-L C C7
+L C-RESCUE-pivi-shield C7
 U 1 1 5496B136
 P 5525 1525
 AR Path="/548ADE5E/5496B136" Ref="C7"  Part="1"
 AR Path="/547008F6/5496B136" Ref="C17"  Part="1"
+AR Path="/5496B136" Ref="C17"  Part="1"
 F 0 "C17" H 5525 1625 40  0000 L CNN
 F 1 "100nF" H 5531 1440 40  0000 L CNN
@@
 $EndComp
 $Comp
-L C C8
+L C-RESCUE-pivi-shield C8
 U 1 1 5496B172
 P 5825 1525
 AR Path="/548ADE5E/5496B172" Ref="C8"  Part="1"
 AR Path="/547008F6/5496B172" Ref="C18"  Part="1"
+AR Path="/5496B172" Ref="C18"  Part="1"
 F 0 "C18" H 5825 1625 40  0000 L CNN
 F 1 "100nF" H 5831 1440 40  0000 L CNN
@@
 $EndComp
 $Comp
-L GND #PWR017
+L GND-RESCUE-pivi-shield #PWR018
 U 1 1 54BF84DA
 P 7400 1800
-F 0 "#PWR017" H 7400 1550 60  0001 C CNN
+F 0 "#PWR018" H 7400 1550 60  0001 C CNN
 F 1 "GND" H 7400 1650 60  0000 C CNN
 F 2 "" H 7400 1800 60  0000 C CNN
@@
 $EndComp
 $Comp
-L GND #PWR018
+L GND-RESCUE-pivi-shield #PWR019
 U 1 1 54BF85B6
 P 7700 1800
-F 0 "#PWR018" H 7700 1550 60  0001 C CNN
+F 0 "#PWR019" H 7700 1550 60  0001 C CNN
 F 1 "GND" H 7700 1650 60  0000 C CNN
 F 2 "" H 7700 1800 60  0000 C CNN
@@
 $EndComp
 $Comp
-L GND #PWR019
+L GND-RESCUE-pivi-shield #PWR020
 U 1 1 54BF87AD
 P 4125 1900
-F 0 "#PWR019" H 4125 1650 60  0001 C CNN
+F 0 "#PWR020" H 4125 1650 60  0001 C CNN
 F 1 "GND" H 4125 1750 60  0000 C CNN
 F 2 "" H 4125 1900 60  0000 C CNN
@@
 $EndComp
 $Comp
-L GND #PWR020
+L GND-RESCUE-pivi-shield #PWR021
 U 1 1 54BF89A3
 P 3325 4900
-F 0 "#PWR020" H 3325 4650 60  0001 C CNN
+F 0 "#PWR021" H 3325 4650 60  0001 C CNN
 F 1 "GND" H 3325 4750 60  0000 C CNN
 F 2 "" H 3325 4900 60  0000 C CNN
@@
 $EndComp
 $Comp
-L GND #PWR021
+L GND-RESCUE-pivi-shield #PWR022
 U 1 1 54BF8BAD
 P 6350 5800
-F 0 "#PWR021" H 6350 5550 60  0001 C CNN
+F 0 "#PWR022" H 6350 5550 60  0001 C CNN
 F 1 "GND" H 6350 5650 60  0000 C CNN
 F 2 "" H 6350 5800 60  0000 C CNN
@@
 	10250 2300 10250 2700
 $Comp
-L GND #PWR022
+L GND-RESCUE-pivi-shield #PWR023
 U 1 1 54BF9940
 P 10450 2700
-F 0 "#PWR022" H 10450 2450 60  0001 C CNN
+F 0 "#PWR023" H 10450 2450 60  0001 C CNN
 F 1 "GND" H 10450 2550 60  0000 C CNN
 F 2 "" H 10450 2700 60  0000 C CNN
@@
 $EndComp
 $Comp
-L PWR_FLAG #FLG023
+L PWR_FLAG #FLG024
 U 1 1 54C23958
 P 4315 6270
-F 0 "#FLG023" H 4315 6365 30  0001 C CNN
+F 0 "#FLG024" H 4315 6365 30  0001 C CNN
 F 1 "PWR_FLAG" H 4315 6450 30  0000 C CNN
 F 2 "" H 4315 6270 60  0000 C CNN
@@
 $EndComp
 $Comp
-L GND #PWR024
+L GND-RESCUE-pivi-shield #PWR025
 U 1 1 54C243B5
 P 4315 7010
-F 0 "#PWR024" H 4315 6760 60  0001 C CNN
+F 0 "#PWR025" H 4315 6760 60  0001 C CNN
 F 1 "GND" H 4315 6860 60  0000 C CNN
 F 2 "" H 4315 7010 60  0000 C CNN
@@
 Text Notes 4460 6910 0    60   ~ 0
 This Inductor should be placed\nnear PIN 60 of the Xmega
+Wire Wire Line
+	4925 2500 5275 2500
+Wire Wire Line
+	5275 2500 5275 2250
+Connection ~ 5275 2250
+Text HLabel 4925 2500 0    60   Input ~ 0
+RESET
 $EndSCHEMATC

Commit message: Fix #4: Move RGB LED from microcontroller to pi.
* Move RGB LED. Now it is controlled by the raspberry pi.
* Change some new libraries for capacitors and resistors.
Parts:
- C1, C10, C2, C4, C5, C6, C7, C8: symbol C-RESCUE-pivi-shield -> C
- C3, C9: symbol CAPAPOL -> C
- X1: symbol CRYSTAL -> Crystal
Changed lines of the file:
@@
 LIBS:txs0104e
 LIBS:less
-LIBS:pivi-shield-cache
 EELAYER 25 0
 EELAYER END
@@
 $EndComp
 $Comp
-L CAPAPOL C3
+L C C3
 U 1 1 546F43CE
 P 4125 1525
@@
 $EndComp
 $Comp
-L C-RESCUE-pivi-shield C4
+L C C4
 U 1 1 548AF338
 P 4600 1525
@@
 $EndComp
 $Comp
-L CAPAPOL C9
+L C C9
 U 1 1 546F43D7
 P 7400 1525
@@
 PF7
 $Comp
-L C-RESCUE-pivi-shield C2
+L C C2
 U 1 1 54863967
 P 3625 4650
@@
 $EndComp
 $Comp
-L CRYSTAL X1
+L Crystal X1
 U 1 1 5486396D
 P 4000 4300
@@
 P 4600 1250
 AR Path="/548ADE5E/548F45ED" Ref="#PWR10"  Part="1"
-AR Path="/547008F6/548F45ED" Ref="#PWR010"  Part="1"
-F 0 "#PWR010" H 4650 1280 20  0001 C CNN
+AR Path="/547008F6/548F45ED" Ref="#PWR09"  Part="1"
+F 0 "#PWR09" H 4650 1280 20  0001 C CNN
 F 1 "+3.3VP" H 4600 1340 30  0000 C CNN
 F 2 "" H 4600 1250 60  0000 C CNN
@@
 P 10000 2150
 AR Path="/548ADE5E/548F468B" Ref="#PWR18"  Part="1"
-AR Path="/547008F6/548F468B" Ref="#PWR011"  Part="1"
-F 0 "#PWR011" H 10050 2180 20  0001 C CNN
+AR Path="/547008F6/548F468B" Ref="#PWR010"  Part="1"
+F 0 "#PWR010" H 10050 2180 20  0001 C CNN
 F 1 "+3.3VP" H 10000 2240 30  0000 C CNN
 F 2 "" H 10000 2150 60  0000 C CNN
@@
 P 8350 3400
 AR Path="/548ADE5E/548F4755" Ref="#PWR16"  Part="1"
-AR Path="/547008F6/548F4755" Ref="#PWR012"  Part="1"
-F 0 "#PWR012" H 8400 3430 20  0001 C CNN
+AR Path="/547008F6/548F4755" Ref="#PWR011"  Part="1"
+F 0 "#PWR011" H 8400 3430 20  0001 C CNN
 F 1 "+3.3VP" H 8350 3490 30  0000 C CNN
 F 2 "" H 8350 3400 60  0000 C CNN
@@
 P 8350 4600
 AR Path="/548ADE5E/548F499C" Ref="#PWR17"  Part="1"
-AR Path="/547008F6/548F499C" Ref="#PWR013"  Part="1"
-F 0 "#PWR013" H 8400 4630 20  0001 C CNN
+AR Path="/547008F6/548F499C" Ref="#PWR012"  Part="1"
+F 0 "#PWR012" H 8400 4630 20  0001 C CNN
 F 1 "+3.3VP" H 8350 4690 30  0000 C CNN
 F 2 "" H 8350 4600 60  0000 C CNN
@@
 $EndComp
 $Comp
-L C-RESCUE-pivi-shield C1
+L C C1
 U 1 1 548F5037
 P 3625 3950
@@
 $EndComp
 $Comp
-L C-RESCUE-pivi-shield C10
+L C C10
 U 1 1 548F53F6
 P 7700 1525
@@
 P 7700 1300
 AR Path="/548ADE5E/548F5520" Ref="#PWR13"  Part="1"
-AR Path="/547008F6/548F5520" Ref="#PWR014"  Part="1"
-F 0 "#PWR014" H 7700 1420 20  0001 C CNN
+AR Path="/547008F6/548F5520" Ref="#PWR013"  Part="1"
+F 0 "#PWR013" H 7700 1420 20  0001 C CNN
 F 1 "+3.3VADC" H 7700 1390 30  0000 C CNN
 F 2 "" H 7700 1300 60  0000 C CNN
@@
 P 8200 2150
 AR Path="/548ADE5E/548F6C6F" Ref="#PWR15"  Part="1"
-AR Path="/547008F6/548F6C6F" Ref="#PWR015"  Part="1"
-F 0 "#PWR015" H 8250 2180 20  0001 C CNN
+AR Path="/547008F6/548F6C6F" Ref="#PWR014"  Part="1"
+F 0 "#PWR014" H 8250 2180 20  0001 C CNN
 F 1 "+3.3VP" H 8200 2240 30  0000 C CNN
 F 2 "" H 8200 2150 60  0000 C CNN
@@
 P 4375 2250
 AR Path="/548ADE5E/5493E84E" Ref="#PWR9"  Part="1"
-AR Path="/547008F6/5493E84E" Ref="#PWR016"  Part="1"
-F 0 "#PWR016" H 4425 2280 20  0001 C CNN
+AR Path="/547008F6/5493E84E" Ref="#PWR015"  Part="1"
+F 0 "#PWR015" H 4425 2280 20  0001 C CNN
 F 1 "+3.3VP" H 4375 2340 30  0000 C CNN
 F 2 "" H 4375 2250 60  0000 C CNN
@@
 P 3450 1300
 AR Path="/548ADE5E/54967597" Ref="#PWR7"  Part="1"
-AR Path="/547008F6/54967597" Ref="#PWR017"  Part="1"
-F 0 "#PWR017" H 3450 1150 60  0001 C CNN
+AR Path="/547008F6/54967597" Ref="#PWR016"  Part="1"
+F 0 "#PWR016" H 3450 1150 60  0001 C CNN
 F 1 "+3V3" H 3450 1440 60  0000 C CNN
 F 2 "" H 3450 1300 60  0000 C CNN
@@
 $EndComp
 $Comp
-L C-RESCUE-pivi-shield C5
+L C C5
 U 1 1 5496B0BB
 P 4925 1525
@@
 $EndComp
 $Comp
-L C-RESCUE-pivi-shield C6
+L C C6
 U 1 1 5496B0F5
 P 5225 1525
@@
 $EndComp
 $Comp
-L C-RESCUE-pivi-shield C7
+L C C7
 U 1 1 5496B136
 P 5525 1525
@@
 $EndComp
 $Comp
-L C-RESCUE-pivi-shield C8
+L C C8
 U 1 1 5496B172
 P 5825 1525
@@
 $EndComp
 $Comp
-L GND-RESCUE-pivi-shield #PWR018
+L GND-RESCUE-pivi-shield #PWR017
 U 1 1 54BF84DA
 P 7400 1800
-F 0 "#PWR018" H 7400 1550 60  0001 C CNN
+F 0 "#PWR017" H 7400 1550 60  0001 C CNN
 F 1 "GND" H 7400 1650 60  0000 C CNN
 F 2 "" H 7400 1800 60  0000 C CNN
@@
 $EndComp
 $Comp
-L GND-RESCUE-pivi-shield #PWR019
+L GND-RESCUE-pivi-shield #PWR018
 U 1 1 54BF85B6
 P 7700 1800
-F 0 "#PWR019" H 7700 1550 60  0001 C CNN
+F 0 "#PWR018" H 7700 1550 60  0001 C CNN
 F 1 "GND" H 7700 1650 60  0000 C CNN
 F 2 "" H 7700 1800 60  0000 C CNN
@@
 $EndComp
 $Comp
-L GND-RESCUE-pivi-shield #PWR020
+L GND-RESCUE-pivi-shield #PWR019
 U 1 1 54BF87AD
 P 4125 1900
-F 0 "#PWR020" H 4125 1650 60  0001 C CNN
+F 0 "#PWR019" H 4125 1650 60  0001 C CNN
 F 1 "GND" H 4125 1750 60  0000 C CNN
 F 2 "" H 4125 1900 60  0000 C CNN
@@
 $EndComp
 $Comp
-L GND-RESCUE-pivi-shield #PWR021
+L GND-RESCUE-pivi-shield #PWR020
 U 1 1 54BF89A3
 P 3325 4900
-F 0 "#PWR021" H 3325 4650 60  0001 C CNN
+F 0 "#PWR020" H 3325 4650 60  0001 C CNN
 F 1 "GND" H 3325 4750 60  0000 C CNN
 F 2 "" H 3325 4900 60  0000 C CNN
@@
 $EndComp
 $Comp
-L GND-RESCUE-pivi-shield #PWR022
+L GND-RESCUE-pivi-shield #PWR021
 U 1 1 54BF8BAD
 P 6350 5800
-F 0 "#PWR022" H 6350 5550 60  0001 C CNN
+F 0 "#PWR021" H 6350 5550 60  0001 C CNN
 F 1 "GND" H 6350 5650 60  0000 C CNN
 F 2 "" H 6350 5800 60  0000 C CNN
@@
 Connection ~ 6350 5625
 Wire Wire Line
-	4125 1300 4125 1325
-Wire Wire Line
-	4125 1725 4125 1900
+	4125 1300 4125 1375
+Wire Wire Line
+	4125 1675 4125 1900
 Wire Wire Line
 	6300 1300 6300 1950
 Connection ~ 4125 1300
 Wire Wire Line
-	4600 1725 4600 1800
-Wire Wire Line
-	4925 1800 4925 1725
-Wire Wire Line
-	5225 1800 5225 1725
-Wire Wire Line
-	5225 1300 5225 1325
-Wire Wire Line
-	4925 1300 4925 1325
-Wire Wire Line
-	4600 1250 4600 1325
+	4600 1675 4600 1800
+Wire Wire Line
+	4925 1675 4925 1800
+Wire Wire Line
+	5225 1675 5225 1800
+Wire Wire Line
+	5225 1300 5225 1375
+Wire Wire Line
+	4925 1300 4925 1375
+Wire Wire Line
+	4600 1250 4600 1375
 Wire Wire Line
 	6500 1300 6500 1950
@@
 	7225 1300 7700 1300
 Wire Wire Line
-	7400 1325 7400 1300
+	7400 1300 7400 1375
 Connection ~ 7400 1300
 Wire Wire Line
-	7400 1725 7400 1800
-Wire Wire Line
-	7700 1725 7700 1800
+	7400 1675 7400 1800
+Wire Wire Line
+	7700 1675 7700 1800
 Wire Wire Line
 	7275 1950 7275 1300
@@
 	9650 2700 10450 2700
 Wire Wire Line
-	5525 1800 5525 1725
-Wire Wire Line
-	5825 1800 5825 1725
-Wire Wire Line
-	5525 1325 5525 1300
+	5525 1675 5525 1800
+Wire Wire Line
+	5825 1675 5825 1800
+Wire Wire Line
+	5525 1300 5525 1375
 Connection ~ 5525 1300
 Wire Wire Line
-	5825 1325 5825 1300
+	5825 1300 5825 1375
 Connection ~ 5825 1300
 Wire Wire Line
@@
 	5000 3800 5350 3800
 Wire Wire Line
-	3825 4650 5350 4650
-Wire Wire Line
-	4000 4600 4000 4650
+	3775 4650 5350 4650
+Wire Wire Line
+	4000 4450 4000 4650
 Connection ~ 4000 4650
 Wire Wire Line
-	3825 3950 4300 3950
-Wire Wire Line
-	4000 3950 4000 4000
+	3775 3950 4300 3950
+Wire Wire Line
+	4000 3950 4000 4150
 Wire Wire Line
 	4300 3950 4300 4550
@@
 Connection ~ 4000 3950
 Wire Wire Line
-	3425 4650 3325 4650
+	3325 4650 3475 4650
 Wire Wire Line
 	3325 3950 3325 4900
 Wire Wire Line
-	3325 3950 3425 3950
+	3325 3950 3475 3950
 Connection ~ 3325 4650
 Wire Wire Line
-	7700 1300 7700 1325
+	7700 1300 7700 1375
 Wire Wire Line
 	5350 2250 4950 2250
@@
 	5350 2950 5000 2950
 Wire Wire Line
-	4125 1800 5825 1800
+	5825 1800 4125 1800
 Connection ~ 4925 1800
 Wire Wire Line
@@
 	10250 2300 10250 2700
 $Comp
-L GND-RESCUE-pivi-shield #PWR023
+L GND-RESCUE-pivi-shield #PWR022
 U 1 1 54BF9940
 P 10450 2700
-F 0 "#PWR023" H 10450 2450 60  0001 C CNN
+F 0 "#PWR022" H 10450 2450 60  0001 C CNN
 F 1 "GND" H 10450 2550 60  0000 C CNN
 F 2 "" H 10450 2700 60  0000 C CNN
@@
 $EndComp
 $Comp
-L PWR_FLAG #FLG024
+L PWR_FLAG #FLG023
 U 1 1 54C23958
 P 4315 6270
-F 0 "#FLG024" H 4315 6365 30  0001 C CNN
+F 0 "#FLG023" H 4315 6365 30  0001 C CNN
 F 1 "PWR_FLAG" H 4315 6450 30  0000 C CNN
 F 2 "" H 4315 6270 60  0000 C CNN
@@
 $EndComp
 $Comp
-L GND-RESCUE-pivi-shield #PWR025
+L GND-RESCUE-pivi-shield #PWR024
 U 1 1 54C243B5
 P 4315 7010
-F 0 "#PWR025" H 4315 6760 60  0001 C CNN
+F 0 "#PWR024" H 4315 6760 60  0001 C CNN
 F 1 "GND" H 4315 6860 60  0000 C CNN
 F 2 "" H 4315 7010 60  0000 C CNN

Commit message: Changing footprints of  audio jack3.5mm Added new footprints. Added debub uart,  reference voltage Added two extra circuits for voltage measure Moving to PIVI 2.0, added circuits for current clamps
Parts:
- removed JP1: JUMPER, Pin_Headers:Pin_Header_Straight_1x02, symbol JUMPER
- C3, C9: symbol C -> CAPAPOL
- R3, R4, R5: symbol R-RESCUE-pivi-shield -> R
- X1: symbol Crystal -> CRYSTAL
- renumbered L1 to L2, L17 to L3
Connections:
- no-connect marks 1 -> 2

Commit message: PCB routed + BOM complete
Parts:
- L3: footprint SMD_Packages:SMD-0603 -> Resistors_SMD:R_0603
Changed lines of the file:
@@
 F 0 "L3" V 4265 6680 40  0000 C CNN
 F 1 "1u" V 4415 6680 40  0000 C CNN
-F 2 "SMD_Packages:SMD-0603" H 4315 6680 60  0001 C CNN
+F 2 "Resistors_SMD:R_0603" H 4315 6680 60  0001 C CNN
 F 3 "" H 4315 6680 60  0000 C CNN
 	1    4315 6680

Commit message: Fix #10: main route not connected.
Right now we have the following power labels:
* +5V from 220v to Raspberry pi and voltage regulator.
* +3V3 from voltage regulator to microcontroller imput and measurement voltage circuit.
* +3.3VP DC digital +3.3v (filter to MCU).
* +3.3VADC DC analog +3.3v
Parts:
- C3, C9: symbol CAPAPOL -> CP
- X1: symbol CRYSTAL -> CRYSTAL_SMD
Connections:
- wire segments 115 -> 116
- no-connect marks 2 -> 3
Changed lines of the file:
@@
 LIBS:txs0104e
 LIBS:less
-LIBS:pivi-shield-cache
 EELAYER 25 0
 EELAYER END
@@
 $EndComp
 $Comp
-L CAPAPOL C3
+L CP C3
 U 1 1 546F43CE
 P 4125 1525
@@
 $EndComp
 $Comp
-L CAPAPOL C9
+L CP C9
 U 1 1 546F43D7
 P 7400 1525
@@
 $EndComp
 $Comp
-L CRYSTAL X1
+L CRYSTAL_SMD X1
 U 1 1 5486396D
 P 4000 4300
@@
 $EndComp
 $Comp
-L +3.3VP #PWR011
+L +3.3VP #PWR013
 U 1 1 548F45ED
 P 4600 1250
-F 0 "#PWR011" H 4650 1280 20  0001 C CNN
+F 0 "#PWR013" H 4650 1280 20  0001 C CNN
 F 1 "+3.3VP" H 4600 1340 30  0000 C CNN
 F 2 "" H 4600 1250 60  0000 C CNN
@@
 $EndComp
 $Comp
-L +3.3VP #PWR012
+L +3.3VP #PWR014
 U 1 1 548F468B
 P 10000 2150
-F 0 "#PWR012" H 10050 2180 20  0001 C CNN
+F 0 "#PWR014" H 10050 2180 20  0001 C CNN
 F 1 "+3.3VP" H 10000 2240 30  0000 C CNN
 F 2 "" H 10000 2150 60  0000 C CNN
@@
 $EndComp
 $Comp
-L +3.3VP #PWR013
+L +3.3VP #PWR015
 U 1 1 548F4755
 P 8350 3400
-F 0 "#PWR013" H 8400 3430 20  0001 C CNN
+F 0 "#PWR015" H 8400 3430 20  0001 C CNN
 F 1 "+3.3VP" H 8350 3490 30  0000 C CNN
 F 2 "" H 8350 3400 60  0000 C CNN
@@
 $EndComp
 $Comp
-L +3.3VP #PWR014
+L +3.3VP #PWR016
 U 1 1 548F499C
 P 8350 4600
-F 0 "#PWR014" H 8400 4630 20  0001 C CNN
+F 0 "#PWR016" H 8400 4630 20  0001 C CNN
 F 1 "+3.3VP" H 8350 4690 30  0000 C CNN
 F 2 "" H 8350 4600 60  0000 C CNN
@@
 $EndComp
 $Comp
-L +3.3VADC #PWR015
+L +3.3VADC #PWR017
 U 1 1 548F5520
 P 7700 1300
-F 0 "#PWR015" H 7700 1420 20  0001 C CNN
+F 0 "#PWR017" H 7700 1420 20  0001 C CNN
 F 1 "+3.3VADC" H 7700 1390 30  0000 C CNN
 F 2 "" H 7700 1300 60  0000 C CNN
@@
 $EndComp
 $Comp
-L +3.3VP #PWR016
+L +3.3VP #PWR018
 U 1 1 5493E84E
 P 4375 2250
-F 0 "#PWR016" H 4425 2280 20  0001 C CNN
+F 0 "#PWR018" H 4425 2280 20  0001 C CNN
 F 1 "+3.3VP" H 4375 2340 30  0000 C CNN
 F 2 "" H 4375 2250 60  0000 C CNN
@@
 $EndComp
 $Comp
-L +3V3 #PWR017
+L +3V3 #PWR019
 U 1 1 54967597
 P 3450 1300
-F 0 "#PWR017" H 3450 1150 60  0001 C CNN
+F 0 "#PWR019" H 3450 1150 60  0001 C CNN
 F 1 "+3V3" H 3450 1440 60  0000 C CNN
 F 2 "" H 3450 1300 60  0000 C CNN
@@
 $EndComp
 $Comp
-L GND #PWR018
+L GND #PWR020
 U 1 1 54BF84DA
 P 7400 1800
-F 0 "#PWR018" H 7400 1550 60  0001 C CNN
+F 0 "#PWR020" H 7400 1550 60  0001 C CNN
 F 1 "GND" H 7400 1650 60  0000 C CNN
 F 2 "" H 7400 1800 60  0000 C CNN
@@
 $EndComp
 $Comp
-L GND #PWR019
+L GND #PWR021
 U 1 1 54BF85B6
 P 7700 1800
-F 0 "#PWR019" H 7700 1550 60  0001 C CNN
+F 0 "#PWR021" H 7700 1550 60  0001 C CNN
 F 1 "GND" H 7700 1650 60  0000 C CNN
 F 2 "" H 7700 1800 60  0000 C CNN
@@
 $EndComp
 $Comp
-L GND #PWR020
+L GND #PWR022
 U 1 1 54BF87AD
 P 4125 1900
-F 0 "#PWR020" H 4125 1650 60  0001 C CNN
+F 0 "#PWR022" H 4125 1650 60  0001 C CNN
 F 1 "GND" H 4125 1750 60  0000 C CNN
 F 2 "" H 4125 1900 60  0000 C CNN
@@
 $EndComp
 $Comp
-L GND #PWR021
+L GND #PWR023
 U 1 1 54BF89A3
 P 3325 4900
-F 0 "#PWR021" H 3325 4650 60  0001 C CNN
+F 0 "#PWR023" H 3325 4650 60  0001 C CNN
 F 1 "GND" H 3325 4750 60  0000 C CNN
 F 2 "" H 3325 4900 60  0000 C CNN
@@
 $EndComp
 $Comp
-L GND #PWR022
+L GND #PWR024
 U 1 1 54BF8BAD
 P 6350 5800
-F 0 "#PWR022" H 6350 5550 60  0001 C CNN
+F 0 "#PWR024" H 6350 5550 60  0001 C CNN
 F 1 "GND" H 6350 5650 60  0000 C CNN
 F 2 "" H 6350 5800 60  0000 C CNN
@@
 $EndComp
 $Comp
-L GND #PWR023
+L GND #PWR025
 U 1 1 54BF9940
 P 10450 2700
-F 0 "#PWR023" H 10450 2450 60  0001 C CNN
+F 0 "#PWR025" H 10450 2450 60  0001 C CNN
 F 1 "GND" H 10450 2550 60  0000 C CNN
 F 2 "" H 10450 2700 60  0000 C CNN
@@
 $EndComp
 $Comp
-L PWR_FLAG #FLG024
+L PWR_FLAG #FLG026
 U 1 1 54C23958
 P 4315 6270
-F 0 "#FLG024" H 4315 6365 30  0001 C CNN
+F 0 "#FLG026" H 4315 6365 30  0001 C CNN
 F 1 "PWR_FLAG" H 4315 6450 30  0000 C CNN
 F 2 "" H 4315 6270 60  0000 C CNN
@@
 $EndComp
 $Comp
-L GND #PWR025
+L GND #PWR027
 U 1 1 54C243B5
 P 4315 7010
-F 0 "#PWR025" H 4315 6760 60  0001 C CNN
+F 0 "#PWR027" H 4315 6760 60  0001 C CNN
 F 1 "GND" H 4315 6860 60  0000 C CNN
 F 2 "" H 4315 7010 60  0000 C CNN
@@
 Connection ~ 6350 5625
 Wire Wire Line
-	4125 1300 4125 1325
-Wire Wire Line
-	4125 1725 4125 1900
+	4125 1300 4125 1375
+Wire Wire Line
+	4125 1675 4125 1900
 Wire Wire Line
 	6300 1300 6300 1950
@@
 	7225 1300 7700 1300
 Wire Wire Line
-	7400 1325 7400 1300
+	7400 1300 7400 1375
 Connection ~ 7400 1300
 Wire Wire Line
-	7400 1725 7400 1800
+	7400 1675 7400 1800
 Wire Wire Line
 	7700 1675 7700 1800
@@
 	3775 4650 5350 4650
 Wire Wire Line
-	4000 4600 4000 4650
+	4000 4500 4000 4650
 Connection ~ 4000 4650
 Wire Wire Line
 	3775 3950 4300 3950
 Wire Wire Line
-	4000 3950 4000 4000
+	4000 3950 4000 4100
 Wire Wire Line
 	4300 3950 4300 4550
@@
 Connection ~ 5275 2250
 NoConn ~ 9150 2600
+Wire Wire Line
+	3900 4300 3850 4300
+NoConn ~ 3850 4300
 $EndSCHEMATC
