File: design/ATXMEGA128A3U.sch (KiCad schematic (older format))
At the start: 19 parts, among them IC1 ATXMEGA128A3U-A, P1 CONN_02X05, X1 32.768kHz +/-20PPM 7pF SMD

Commit message: Fix #7, Fix #8, Fix #9, Fix #10, Fix #11
Several fixes improvements:
* Fix #7: Add 2mm idle to each side of the connector.
* Fix #8: Add 0.25mm to each side of the connector.
* Fix #9: Mirror component. Checked with the datasheet.
* Fix #10: correct label name.
* Fix #11: Changed the terminal block for one with a better mouting system.

Also check the Raspberry pi 20 pin header. It is place in the correct position.
Parts:
- P1: value CONN_02X05 -> JTAG connector
- X1: symbol CRYSTAL_SMD -> Crystal
Connections:
- wire segments 116 -> 115
- no-connect marks 3 -> 2
Changed lines of the file:
@@
 $EndComp
 $Comp
-L CRYSTAL_SMD X1
+L Crystal X1
 U 1 1 5486396D
 P 4000 4300
@@
 P 9400 2500
 F 0 "P1" H 9400 2800 50  0000 C CNN
-F 1 "CONN_02X05" H 9400 2200 50  0000 C CNN
+F 1 "JTAG connector" H 9400 2200 50  0000 C CNN
 F 2 "Pin_Headers:Pin_Header_Straight_2x05" H 9400 2125 60  0000 C CNN
 F 3 "" H 9400 1300 60  0000 C CNN
@@
 	3775 4650 5350 4650
 Wire Wire Line
-	4000 4500 4000 4650
+	4000 4450 4000 4650
 Connection ~ 4000 4650
 Wire Wire Line
 	3775 3950 4300 3950
 Wire Wire Line
-	4000 3950 4000 4100
+	4000 3950 4000 4150
 Wire Wire Line
 	4300 3950 4300 4550
@@
 Connection ~ 5275 2250
 NoConn ~ 9150 2600
-Wire Wire Line
-	3900 4300 3850 4300
-NoConn ~ 3850 4300
 $EndSCHEMATC
