File: design/voltage.sch (KiCad schematic (older format))
At the start: 12 parts

Commit message: Starting PIVI 2.0 * sch ready. * components in PCB placed.
Changed lines of the file:
@@
 AR Path="/548DF2C8/55B9EDA2/5497B2D6" Ref="R44"  Part="1"
 AR Path="/548DF2C8/55BA09A0/5497B2D6" Ref="R51"  Part="1"
-F 0 "R19" V 6265 4235 40  0000 C CNN
+F 0 "R51" V 6265 4235 40  0000 C CNN
 F 1 "10k" V 6192 4236 40  0000 C CNN
 F 2 "Resistors_SMD:R_0603" V 6115 4235 30  0000 C CNN
@@
 AR Path="/548DF2C8/55B9EDA2/5497B2DD" Ref="R45"  Part="1"
 AR Path="/548DF2C8/55BA09A0/5497B2DD" Ref="R52"  Part="1"
-F 0 "R20" V 6990 3835 40  0000 C CNN
+F 0 "R52" V 6990 3835 40  0000 C CNN
 F 1 "100" V 6917 3836 40  0000 C CNN
 F 2 "Resistors_SMD:R_0603" V 6810 3835 30  0000 C CNN
@@
 AR Path="/548DF2C8/55B9EDA2/5497B2E4" Ref="C24"  Part="1"
 AR Path="/548DF2C8/55BA09A0/5497B2E4" Ref="C27"  Part="1"
-F 0 "C15" H 6860 3210 40  0000 L CNN
+F 0 "C27" H 6860 3210 40  0000 L CNN
 F 1 "100n" H 6866 3025 40  0000 L CNN
 F 2 "Capacitors_SMD:C_0603" H 7085 3360 30  0000 C CNN
@@
 AR Path="/548DF2C8/55B9EDA2/5497B2EB" Ref="C25"  Part="1"
 AR Path="/548DF2C8/55BA09A0/5497B2EB" Ref="C28"  Part="1"
-F 0 "C16" H 7835 4235 40  0000 L CNN
+F 0 "C28" H 7835 4235 40  0000 L CNN
 F 1 "330nF" H 7860 4160 40  0000 L CNN
 F 2 "Capacitors_SMD:C_0603" V 7585 4235 30  0000 C CNN
@@
 AR Path="/548DF2C8/55B9EDA2/5497B2FF" Ref="R47"  Part="1"
 AR Path="/548DF2C8/55BA09A0/5497B2FF" Ref="R54"  Part="1"
-F 0 "R22" V 7210 4235 40  0000 C CNN
+F 0 "R54" V 7210 4235 40  0000 C CNN
 F 1 "10k" V 7292 4236 40  0000 C CNN
 F 2 "Resistors_SMD:R_0603" V 7360 4235 30  0000 C CNN
@@
 AR Path="/548DF2C8/55B9EDA2/548E33DD" Ref="R41"  Part="1"
 AR Path="/548DF2C8/55BA09A0/548E33DD" Ref="R48"  Part="1"
-F 0 "R16" V 4840 3835 40  0000 C CNN
+F 0 "R48" V 4840 3835 40  0000 C CNN
 F 1 "220k" V 4767 3836 40  0000 C CNN
 F 2 "Resistors_SMD:R_2512" V 4660 3835 30  0000 C CNN
@@
 AR Path="/548DF2C8/55B9EDA2/548E40C9" Ref="R46"  Part="1"
 AR Path="/548DF2C8/55BA09A0/548E40C9" Ref="R53"  Part="1"
-F 0 "R21" V 7210 3510 40  0000 C CNN
+F 0 "R53" V 7210 3510 40  0000 C CNN
 F 1 "10k" V 7292 3511 40  0000 C CNN
 F 2 "Resistors_SMD:R_0603" V 7360 3510 30  0000 C CNN
@@
 AR Path="/548DF2C8/55B9EDA2/548DF4C0" Ref="R42"  Part="1"
 AR Path="/548DF2C8/55BA09A0/548DF4C0" Ref="R49"  Part="1"
-F 0 "R17" V 5390 3835 40  0000 C CNN
+F 0 "R49" V 5390 3835 40  0000 C CNN
 F 1 "220k" V 5317 3836 40  0000 C CNN
 F 2 "Resistors_SMD:R_2512" V 5210 3835 30  0000 C CNN
@@
 AR Path="/548DF2C8/55B9EDA2/548DF506" Ref="R43"  Part="1"
 AR Path="/548DF2C8/55BA09A0/548DF506" Ref="R50"  Part="1"
-F 0 "R18" V 5940 3835 40  0000 C CNN
+F 0 "R50" V 5940 3835 40  0000 C CNN
 F 1 "220k" V 5867 3836 40  0000 C CNN
 F 2 "Resistors_SMD:R_2512" V 5760 3835 30  0000 C CNN
@@
 AR Path="/548DF2C8/55B9EDA2/54BDE7C8" Ref="L9"  Part="1"
 AR Path="/548DF2C8/55BA09A0/54BDE7C8" Ref="L11"  Part="1"
-F 0 "L7" V 6410 2910 40  0000 C CNN
+F 0 "L11" V 6410 2910 40  0000 C CNN
 F 1 "1u" V 6560 2910 40  0000 C CNN
 F 2 "SMD_Packages:SMD-0603" V 6335 3235 60  0000 C CNN
@@
 $EndComp
 $Comp
-L +3V3 #PWR49
+L +3V3 #PWR054
 U 1 1 54BE015B
 P 6160 2810
-AR Path="/548DF2C8/55B216B6/54BE015B" Ref="#PWR49"  Part="1"
-AR Path="/548DF2C8/55B9EDA2/54BE015B" Ref="#PWR64"  Part="1"
-AR Path="/548DF2C8/55BA09A0/54BE015B" Ref="#PWR67"  Part="1"
-F 0 "#PWR49" H 6160 2660 60  0001 C CNN
+AR Path="/548DF2C8/55B216B6/54BE015B" Ref="#PWR054"  Part="1"
+AR Path="/548DF2C8/55B9EDA2/54BE015B" Ref="#PWR069"  Part="1"
+AR Path="/548DF2C8/55BA09A0/54BE015B" Ref="#PWR072"  Part="1"
+F 0 "#PWR072" H 6160 2660 60  0001 C CNN
 F 1 "+3V3" H 6160 2950 60  0000 C CNN
 F 2 "" H 6160 2810 60  0000 C CNN
@@
 $EndComp
 $Comp
-L GND #PWR50
+L GND #PWR055
 U 1 1 54C00611
 P 6860 3360
-AR Path="/548DF2C8/55B216B6/54C00611" Ref="#PWR50"  Part="1"
-AR Path="/548DF2C8/55B9EDA2/54C00611" Ref="#PWR65"  Part="1"
-AR Path="/548DF2C8/55BA09A0/54C00611" Ref="#PWR68"  Part="1"
-F 0 "#PWR50" H 6860 3110 60  0001 C CNN
+AR Path="/548DF2C8/55B216B6/54C00611" Ref="#PWR055"  Part="1"
+AR Path="/548DF2C8/55B9EDA2/54C00611" Ref="#PWR070"  Part="1"
+AR Path="/548DF2C8/55BA09A0/54C00611" Ref="#PWR073"  Part="1"
+F 0 "#PWR073" H 6860 3110 60  0001 C CNN
 F 1 "GND" H 6860 3210 60  0000 C CNN
 F 2 "" H 6860 3360 60  0000 C CNN
@@
 $EndComp
 $Comp
-L GND #PWR51
+L GND #PWR056
 U 1 1 54C006EB
 P 7285 4685
-AR Path="/548DF2C8/55B216B6/54C006EB" Ref="#PWR51"  Part="1"
-AR Path="/548DF2C8/55B9EDA2/54C006EB" Ref="#PWR66"  Part="1"
-AR Path="/548DF2C8/55BA09A0/54C006EB" Ref="#PWR69"  Part="1"
-F 0 "#PWR51" H 7285 4435 60  0001 C CNN
+AR Path="/548DF2C8/55B216B6/54C006EB" Ref="#PWR056"  Part="1"
+AR Path="/548DF2C8/55B9EDA2/54C006EB" Ref="#PWR071"  Part="1"
+AR Path="/548DF2C8/55BA09A0/54C006EB" Ref="#PWR074"  Part="1"
+F 0 "#PWR074" H 7285 4435 60  0001 C CNN
 F 1 "GND" H 7285 4535 60  0000 C CNN
 F 2 "" H 7285 4685 60  0000 C CNN
@@
 AR Path="/548DF2C8/55B9EDA2/54C1942B" Ref="C23"  Part="1"
 AR Path="/548DF2C8/55BA09A0/54C1942B" Ref="C26"  Part="1"
-F 0 "C14" V 6535 3910 50  0000 L CNN
+F 0 "C26" V 6535 3910 50  0000 L CNN
 F 1 "33uF" V 6610 3910 50  0000 L CNN
 F 2 "Capacitors_SMD:C_0805" V 6310 3835 30  0000 C CNN
@@
 AR Path="/548DF2C8/55B9EDA2/548E4464" Ref="L8"  Part="1"
 AR Path="/548DF2C8/55BA09A0/548E4464" Ref="L10"  Part="1"
-F 0 "L6" V 4125 3835 40  0000 C CNN
+F 0 "L10" V 4125 3835 40  0000 C CNN
 F 1 "1uH" V 4275 3835 40  0000 C CNN
 F 2 "Inductors_NEOSID:Neosid_Inductor_SM-NE30_SMD1210" V 4375 3860 60  0000 C CNN

Commit message: PCB routed + BOM complete
Parts:
- L7: footprint SMD_Packages:SMD-0603 -> Resistors_SMD:R_0603
Changed lines of the file:
@@
 AR Path="/548DF2C8/55B9EDA2/5497B2D6" Ref="R44"  Part="1"
 AR Path="/548DF2C8/55BA09A0/5497B2D6" Ref="R51"  Part="1"
-F 0 "R51" V 6265 4235 40  0000 C CNN
+F 0 "R19" V 6265 4235 40  0000 C CNN
 F 1 "10k" V 6192 4236 40  0000 C CNN
 F 2 "Resistors_SMD:R_0603" V 6115 4235 30  0000 C CNN
@@
 AR Path="/548DF2C8/55B9EDA2/5497B2DD" Ref="R45"  Part="1"
 AR Path="/548DF2C8/55BA09A0/5497B2DD" Ref="R52"  Part="1"
-F 0 "R52" V 6990 3835 40  0000 C CNN
+F 0 "R20" V 6990 3835 40  0000 C CNN
 F 1 "100" V 6917 3836 40  0000 C CNN
 F 2 "Resistors_SMD:R_0603" V 6810 3835 30  0000 C CNN
@@
 AR Path="/548DF2C8/55B9EDA2/5497B2E4" Ref="C24"  Part="1"
 AR Path="/548DF2C8/55BA09A0/5497B2E4" Ref="C27"  Part="1"
-F 0 "C27" H 6860 3210 40  0000 L CNN
+F 0 "C15" H 6860 3210 40  0000 L CNN
 F 1 "100n" H 6866 3025 40  0000 L CNN
 F 2 "Capacitors_SMD:C_0603" H 7085 3360 30  0000 C CNN
@@
 AR Path="/548DF2C8/55B9EDA2/5497B2EB" Ref="C25"  Part="1"
 AR Path="/548DF2C8/55BA09A0/5497B2EB" Ref="C28"  Part="1"
-F 0 "C28" H 7835 4235 40  0000 L CNN
+F 0 "C16" H 7835 4235 40  0000 L CNN
 F 1 "330nF" H 7860 4160 40  0000 L CNN
 F 2 "Capacitors_SMD:C_0603" V 7585 4235 30  0000 C CNN
@@
 AR Path="/548DF2C8/55B9EDA2/5497B2FF" Ref="R47"  Part="1"
 AR Path="/548DF2C8/55BA09A0/5497B2FF" Ref="R54"  Part="1"
-F 0 "R54" V 7210 4235 40  0000 C CNN
+F 0 "R22" V 7210 4235 40  0000 C CNN
 F 1 "10k" V 7292 4236 40  0000 C CNN
 F 2 "Resistors_SMD:R_0603" V 7360 4235 30  0000 C CNN
@@
 AR Path="/548DF2C8/55B9EDA2/548E33DD" Ref="R41"  Part="1"
 AR Path="/548DF2C8/55BA09A0/548E33DD" Ref="R48"  Part="1"
-F 0 "R48" V 4840 3835 40  0000 C CNN
+F 0 "R16" V 4840 3835 40  0000 C CNN
 F 1 "220k" V 4767 3836 40  0000 C CNN
 F 2 "Resistors_SMD:R_2512" V 4660 3835 30  0000 C CNN
@@
 AR Path="/548DF2C8/55B9EDA2/548E40C9" Ref="R46"  Part="1"
 AR Path="/548DF2C8/55BA09A0/548E40C9" Ref="R53"  Part="1"
-F 0 "R53" V 7210 3510 40  0000 C CNN
+F 0 "R21" V 7210 3510 40  0000 C CNN
 F 1 "10k" V 7292 3511 40  0000 C CNN
 F 2 "Resistors_SMD:R_0603" V 7360 3510 30  0000 C CNN
@@
 AR Path="/548DF2C8/55B9EDA2/548DF4C0" Ref="R42"  Part="1"
 AR Path="/548DF2C8/55BA09A0/548DF4C0" Ref="R49"  Part="1"
-F 0 "R49" V 5390 3835 40  0000 C CNN
+F 0 "R17" V 5390 3835 40  0000 C CNN
 F 1 "220k" V 5317 3836 40  0000 C CNN
 F 2 "Resistors_SMD:R_2512" V 5210 3835 30  0000 C CNN
@@
 AR Path="/548DF2C8/55B9EDA2/548DF506" Ref="R43"  Part="1"
 AR Path="/548DF2C8/55BA09A0/548DF506" Ref="R50"  Part="1"
-F 0 "R50" V 5940 3835 40  0000 C CNN
+F 0 "R18" V 5940 3835 40  0000 C CNN
 F 1 "220k" V 5867 3836 40  0000 C CNN
 F 2 "Resistors_SMD:R_2512" V 5760 3835 30  0000 C CNN
@@
 AR Path="/548DF2C8/55B9EDA2/54BDE7C8" Ref="L9"  Part="1"
 AR Path="/548DF2C8/55BA09A0/54BDE7C8" Ref="L11"  Part="1"
-F 0 "L11" V 6410 2910 40  0000 C CNN
+F 0 "L7" V 6410 2910 40  0000 C CNN
 F 1 "1u" V 6560 2910 40  0000 C CNN
-F 2 "SMD_Packages:SMD-0603" V 6335 3235 60  0000 C CNN
+F 2 "Resistors_SMD:R_0603" V 6335 3235 60  0000 C CNN
 F 3 "" H 6460 2910 60  0000 C CNN
 	1    6460 2910
@@
 AR Path="/548DF2C8/55B9EDA2/54BE015B" Ref="#PWR069"  Part="1"
 AR Path="/548DF2C8/55BA09A0/54BE015B" Ref="#PWR072"  Part="1"
-F 0 "#PWR072" H 6160 2660 60  0001 C CNN
+F 0 "#PWR054" H 6160 2660 60  0001 C CNN
 F 1 "+3V3" H 6160 2950 60  0000 C CNN
 F 2 "" H 6160 2810 60  0000 C CNN
@@
 AR Path="/548DF2C8/55B9EDA2/54C00611" Ref="#PWR070"  Part="1"
 AR Path="/548DF2C8/55BA09A0/54C00611" Ref="#PWR073"  Part="1"
-F 0 "#PWR073" H 6860 3110 60  0001 C CNN
+F 0 "#PWR055" H 6860 3110 60  0001 C CNN
 F 1 "GND" H 6860 3210 60  0000 C CNN
 F 2 "" H 6860 3360 60  0000 C CNN
@@
 AR Path="/548DF2C8/55B9EDA2/54C006EB" Ref="#PWR071"  Part="1"
 AR Path="/548DF2C8/55BA09A0/54C006EB" Ref="#PWR074"  Part="1"
-F 0 "#PWR074" H 7285 4435 60  0001 C CNN
+F 0 "#PWR056" H 7285 4435 60  0001 C CNN
 F 1 "GND" H 7285 4535 60  0000 C CNN
 F 2 "" H 7285 4685 60  0000 C CNN
@@
 AR Path="/548DF2C8/55B9EDA2/54C1942B" Ref="C23"  Part="1"
 AR Path="/548DF2C8/55BA09A0/54C1942B" Ref="C26"  Part="1"
-F 0 "C26" V 6535 3910 50  0000 L CNN
+F 0 "C14" V 6535 3910 50  0000 L CNN
 F 1 "33uF" V 6610 3910 50  0000 L CNN
 F 2 "Capacitors_SMD:C_0805" V 6310 3835 30  0000 C CNN
@@
 AR Path="/548DF2C8/55B9EDA2/548E4464" Ref="L8"  Part="1"
 AR Path="/548DF2C8/55BA09A0/548E4464" Ref="L10"  Part="1"
-F 0 "L10" V 4125 3835 40  0000 C CNN
+F 0 "L6" V 4125 3835 40  0000 C CNN
 F 1 "1uH" V 4275 3835 40  0000 C CNN
 F 2 "Inductors_NEOSID:Neosid_Inductor_SM-NE30_SMD1210" V 4375 3860 60  0000 C CNN

Commit message: Fix #10: main route not connected.
Right now we have the following power labels:
* +5V from 220v to Raspberry pi and voltage regulator.
* +3V3 from voltage regulator to microcontroller imput and measurement voltage circuit.
* +3.3VP DC digital +3.3v (filter to MCU).
* +3.3VADC DC analog +3.3v
Changed lines of the file:
@@
 LIBS:txs0104e
 LIBS:less
-LIBS:pivi-shield-cache
 EELAYER 25 0
 EELAYER END
@@
 AR Path="/548DF2C8/55B9EDA2/5497B2D6" Ref="R44"  Part="1"
 AR Path="/548DF2C8/55BA09A0/5497B2D6" Ref="R51"  Part="1"
-F 0 "R19" V 6265 4235 40  0000 C CNN
+F 0 "R51" V 6265 4235 40  0000 C CNN
 F 1 "10k" V 6192 4236 40  0000 C CNN
 F 2 "Resistors_SMD:R_0603" V 6115 4235 30  0000 C CNN
@@
 AR Path="/548DF2C8/55B9EDA2/5497B2DD" Ref="R45"  Part="1"
 AR Path="/548DF2C8/55BA09A0/5497B2DD" Ref="R52"  Part="1"
-F 0 "R20" V 6990 3835 40  0000 C CNN
+F 0 "R52" V 6990 3835 40  0000 C CNN
 F 1 "100" V 6917 3836 40  0000 C CNN
 F 2 "Resistors_SMD:R_0603" V 6810 3835 30  0000 C CNN
@@
 AR Path="/548DF2C8/55B9EDA2/5497B2E4" Ref="C24"  Part="1"
 AR Path="/548DF2C8/55BA09A0/5497B2E4" Ref="C27"  Part="1"
-F 0 "C15" H 6860 3210 40  0000 L CNN
+F 0 "C27" H 6860 3210 40  0000 L CNN
 F 1 "100n" H 6866 3025 40  0000 L CNN
 F 2 "Capacitors_SMD:C_0603" H 7085 3360 30  0000 C CNN
@@
 AR Path="/548DF2C8/55B9EDA2/5497B2EB" Ref="C25"  Part="1"
 AR Path="/548DF2C8/55BA09A0/5497B2EB" Ref="C28"  Part="1"
-F 0 "C16" H 7835 4235 40  0000 L CNN
+F 0 "C28" H 7835 4235 40  0000 L CNN
 F 1 "330nF" H 7860 4160 40  0000 L CNN
 F 2 "Capacitors_SMD:C_0603" V 7585 4235 30  0000 C CNN
@@
 AR Path="/548DF2C8/55B9EDA2/5497B2FF" Ref="R47"  Part="1"
 AR Path="/548DF2C8/55BA09A0/5497B2FF" Ref="R54"  Part="1"
-F 0 "R22" V 7210 4235 40  0000 C CNN
+F 0 "R54" V 7210 4235 40  0000 C CNN
 F 1 "10k" V 7292 4236 40  0000 C CNN
 F 2 "Resistors_SMD:R_0603" V 7360 4235 30  0000 C CNN
@@
 AR Path="/548DF2C8/55B9EDA2/548E33DD" Ref="R41"  Part="1"
 AR Path="/548DF2C8/55BA09A0/548E33DD" Ref="R48"  Part="1"
-F 0 "R16" V 4840 3835 40  0000 C CNN
+F 0 "R48" V 4840 3835 40  0000 C CNN
 F 1 "220k" V 4767 3836 40  0000 C CNN
 F 2 "Resistors_SMD:R_2512" V 4660 3835 30  0000 C CNN
@@
 AR Path="/548DF2C8/55B9EDA2/548E40C9" Ref="R46"  Part="1"
 AR Path="/548DF2C8/55BA09A0/548E40C9" Ref="R53"  Part="1"
-F 0 "R21" V 7210 3510 40  0000 C CNN
+F 0 "R53" V 7210 3510 40  0000 C CNN
 F 1 "10k" V 7292 3511 40  0000 C CNN
 F 2 "Resistors_SMD:R_0603" V 7360 3510 30  0000 C CNN
@@
 AR Path="/548DF2C8/55B9EDA2/548DF4C0" Ref="R42"  Part="1"
 AR Path="/548DF2C8/55BA09A0/548DF4C0" Ref="R49"  Part="1"
-F 0 "R17" V 5390 3835 40  0000 C CNN
+F 0 "R49" V 5390 3835 40  0000 C CNN
 F 1 "220k" V 5317 3836 40  0000 C CNN
 F 2 "Resistors_SMD:R_2512" V 5210 3835 30  0000 C CNN
@@
 AR Path="/548DF2C8/55B9EDA2/548DF506" Ref="R43"  Part="1"
 AR Path="/548DF2C8/55BA09A0/548DF506" Ref="R50"  Part="1"
-F 0 "R18" V 5940 3835 40  0000 C CNN
+F 0 "R50" V 5940 3835 40  0000 C CNN
 F 1 "220k" V 5867 3836 40  0000 C CNN
 F 2 "Resistors_SMD:R_2512" V 5760 3835 30  0000 C CNN
@@
 AR Path="/548DF2C8/55B9EDA2/54BDE7C8" Ref="L9"  Part="1"
 AR Path="/548DF2C8/55BA09A0/54BDE7C8" Ref="L11"  Part="1"
-F 0 "L7" V 6410 2910 40  0000 C CNN
+F 0 "L11" V 6410 2910 40  0000 C CNN
 F 1 "1u" V 6560 2910 40  0000 C CNN
 F 2 "Resistors_SMD:R_0603" V 6335 3235 60  0000 C CNN
@@
 $EndComp
 $Comp
-L +3V3 #PWR054
+L +3V3 #PWR056
 U 1 1 54BE015B
 P 6160 2810
-AR Path="/548DF2C8/55B216B6/54BE015B" Ref="#PWR054"  Part="1"
-AR Path="/548DF2C8/55B9EDA2/54BE015B" Ref="#PWR069"  Part="1"
-AR Path="/548DF2C8/55BA09A0/54BE015B" Ref="#PWR072"  Part="1"
-F 0 "#PWR054" H 6160 2660 60  0001 C CNN
+AR Path="/548DF2C8/55B216B6/54BE015B" Ref="#PWR056"  Part="1"
+AR Path="/548DF2C8/55B9EDA2/54BE015B" Ref="#PWR071"  Part="1"
+AR Path="/548DF2C8/55BA09A0/54BE015B" Ref="#PWR074"  Part="1"
+F 0 "#PWR074" H 6160 2660 60  0001 C CNN
 F 1 "+3V3" H 6160 2950 60  0000 C CNN
 F 2 "" H 6160 2810 60  0000 C CNN
@@
 $EndComp
 $Comp
-L GND #PWR055
+L GND #PWR057
 U 1 1 54C00611
 P 6860 3360
-AR Path="/548DF2C8/55B216B6/54C00611" Ref="#PWR055"  Part="1"
-AR Path="/548DF2C8/55B9EDA2/54C00611" Ref="#PWR070"  Part="1"
-AR Path="/548DF2C8/55BA09A0/54C00611" Ref="#PWR073"  Part="1"
-F 0 "#PWR055" H 6860 3110 60  0001 C CNN
+AR Path="/548DF2C8/55B216B6/54C00611" Ref="#PWR057"  Part="1"
+AR Path="/548DF2C8/55B9EDA2/54C00611" Ref="#PWR072"  Part="1"
+AR Path="/548DF2C8/55BA09A0/54C00611" Ref="#PWR075"  Part="1"
+F 0 "#PWR075" H 6860 3110 60  0001 C CNN
 F 1 "GND" H 6860 3210 60  0000 C CNN
 F 2 "" H 6860 3360 60  0000 C CNN
@@
 $EndComp
 $Comp
-L GND #PWR056
+L GND #PWR058
 U 1 1 54C006EB
 P 7285 4685
-AR Path="/548DF2C8/55B216B6/54C006EB" Ref="#PWR056"  Part="1"
-AR Path="/548DF2C8/55B9EDA2/54C006EB" Ref="#PWR071"  Part="1"
-AR Path="/548DF2C8/55BA09A0/54C006EB" Ref="#PWR074"  Part="1"
-F 0 "#PWR056" H 7285 4435 60  0001 C CNN
+AR Path="/548DF2C8/55B216B6/54C006EB" Ref="#PWR058"  Part="1"
+AR Path="/548DF2C8/55B9EDA2/54C006EB" Ref="#PWR073"  Part="1"
+AR Path="/548DF2C8/55BA09A0/54C006EB" Ref="#PWR076"  Part="1"
+F 0 "#PWR076" H 7285 4435 60  0001 C CNN
 F 1 "GND" H 7285 4535 60  0000 C CNN
 F 2 "" H 7285 4685 60  0000 C CNN
@@
 AR Path="/548DF2C8/55B9EDA2/54C1942B" Ref="C23"  Part="1"
 AR Path="/548DF2C8/55BA09A0/54C1942B" Ref="C26"  Part="1"
-F 0 "C14" V 6535 3910 50  0000 L CNN
+F 0 "C26" V 6535 3910 50  0000 L CNN
 F 1 "33uF" V 6610 3910 50  0000 L CNN
 F 2 "Capacitors_SMD:C_0805" V 6310 3835 30  0000 C CNN
@@
 AR Path="/548DF2C8/55B9EDA2/548E4464" Ref="L8"  Part="1"
 AR Path="/548DF2C8/55BA09A0/548E4464" Ref="L10"  Part="1"
-F 0 "L6" V 4125 3835 40  0000 C CNN
+F 0 "L10" V 4125 3835 40  0000 C CNN
 F 1 "1uH" V 4275 3835 40  0000 C CNN
 F 2 "Inductors_NEOSID:Neosid_Inductor_SM-NE30_SMD1210" V 4375 3860 60  0000 C CNN
